Commit message: add tr for /odom /base_laser_link /camera_link

File: moonbuggy_ros/urdf/moonbuggy.urdf.xacro (robot description, xacro)
@@ -149,3 +149,21 @@
     <origin xyz="${mount_spacing} 0 0" />
   </joint>
+  <link name="odom"></link>
+  <joint name="odom_joint" type="fixed">
+    <parent link="mid_mount"/>
+    <child link="odom"/>
+    <origin xyz="0 0 0"/>
+  </joint>
+  <link name="base_laser_link"></link>
+  <joint name="base_laser_link_joint" type="fixed">
+    <parent link="mid_mount"/>
+    <child link="base_laser_link"/>
+    <origin xyz="0.05 0 0.1"/>
+  </joint>
+  <link name="camera_link"></link>
+  <joint name="camera_link_joint" type="fixed">
+    <parent link="mid_mount"/>
+    <child link="camera_link"/>
+    <origin xyz="0.05 0 0.1"/>
+  </joint>
 </robot>

Commit message: remove incorrect tf for odom

File: moonbuggy_ros/urdf/moonbuggy.urdf.xacro (robot description, xacro)
@@ -149,10 +149,4 @@
     <origin xyz="${mount_spacing} 0 0" />
   </joint>
-  <link name="odom"></link>
-  <joint name="odom_joint" type="fixed">
-    <parent link="mid_mount"/>
-    <child link="odom"/>
-    <origin xyz="0 0 0"/>
-  </joint>
   <link name="base_laser_link"></link>
   <joint name="base_laser_link_joint" type="fixed">

Commit message: slam bring-up draft 2

File: moonbuggy_ros/urdf/moonbuggy.urdf.xacro (robot description, xacro)
@@ -161,3 +161,15 @@
     <origin xyz="0.05 0 0.1"/>
   </joint>
+  <link name="map"></link>
+  <joint name="map_link_joint" type="fixed">
+    <parent link="mid_mount"/>
+    <child link="map"/>
+    <origin xyz="0 0 0"/>
+  </joint>
+  <link name="base_footprint"></link>
+  <joint name="base_footprint_link_joint" type="fixed">
+    <parent link="mid_mount"/>
+    <child link="base_footprint"/>
+    <origin xyz="0 0 0"/>
+  </joint>
 </robot>
